Commit message: Adds cameras

File: yumi.urdf (robot description, URDF)
Before this commit: robot yumi, 24 links, 24 joints
Links:
- added link gripper_l_center
- added link left_camera, mass 0.1; collision box size=0.025 0.090 0.025; visual mesh filename=package://yumi_description/meshes/camera/d435.dae
- added link right_camera, mass 0.1; collision box size=0.025 0.090 0.025; visual mesh filename=package://yumi_description/meshes/camera/d435.dae
Joints:
- added joint left_camera_joint: type fixed, parent gripper_l_base, child left_camera, origin xyz=0.08 0.0 0.03 rpy=0 -1.57 3.141592653589793
- added joint right_camera_joint: type fixed, parent gripper_r_base, child right_camera, origin xyz=0.08 0.0 0.03 rpy=0 -1.57 3.141592653589793
- joint gripper_r_joint_m: mimic joint=gripper_r_joint -> (none)
